File: hardware/Rev2/ChargePump.sch (KiCad schematic (older format))
At the start: 8 parts

Commit message: created PCB and gerbers
Parts:
- C1, C2, C3: renamed from C?; footprint (none) -> Capacitors_SMD:C_0805_HandSoldering
- D1, D2, D3: renamed from D?; footprint (none) -> Diodes_SMD:D_SOD-123
- R1, R2: renamed from R?; footprint (none) -> Resistors_SMD:R_0603_HandSoldering
Changed lines of the file:
@@
 LIBS:contrib
 LIBS:valves
+LIBS:PWM10-cache
 EELAYER 25 0
 EELAYER END
 $Descr A4 11693 8268
 encoding utf-8
-Sheet 2 5
+Sheet 2 7
 Title ""
 Date ""
@@
 $EndDescr
 $Comp
-L D_Small D?
+L D_Small D1
 U 1 1 592363A2
 P 5425 3400
-F 0 "D?" H 5375 3480 50  0000 L CNN
+F 0 "D1" H 5375 3480 50  0000 L CNN
 F 1 "D_Small" H 5275 3320 50  0000 L CNN
-F 2 "" V 5425 3400 50  0000 C CNN
+F 2 "Diodes_SMD:D_SOD-123" V 5425 3400 50  0001 C CNN
 F 3 "" V 5425 3400 50  0000 C CNN
 	1    5425 3400
@@
 $EndComp
 $Comp
-L D_Small D?
+L D_Small D2
 U 1 1 59236465
 P 5750 3400
-F 0 "D?" H 5700 3480 50  0000 L CNN
+F 0 "D2" H 5700 3480 50  0000 L CNN
 F 1 "D_Small" H 5600 3320 50  0000 L CNN
-F 2 "" V 5750 3400 50  0000 C CNN
+F 2 "Diodes_SMD:D_SOD-123" V 5750 3400 50  0001 C CNN
 F 3 "" V 5750 3400 50  0000 C CNN
 	1    5750 3400
@@
 $EndComp
 $Comp
-L D_Small D?
+L D_Small D3
 U 1 1 592364A3
 P 6075 3400
-F 0 "D?" H 6025 3480 50  0000 L CNN
+F 0 "D3" H 6025 3480 50  0000 L CNN
 F 1 "D_Small" H 5925 3320 50  0000 L CNN
-F 2 "" V 6075 3400 50  0000 C CNN
+F 2 "Diodes_SMD:D_SOD-123" V 6075 3400 50  0001 C CNN
 F 3 "" V 6075 3400 50  0000 C CNN
 	1    6075 3400
@@
 	6175 3400 6425 3400
 $Comp
-L C_Small C?
+L C_Small C3
 U 1 1 592364EC
 P 6325 3575
-F 0 "C?" H 6335 3645 50  0000 L CNN
+F 0 "C3" H 6335 3645 50  0000 L CNN
 F 1 "1uF" H 6335 3495 50  0000 L CNN
-F 2 "" H 6325 3575 50  0000 C CNN
+F 2 "Capacitors_SMD:C_0805_HandSoldering" H 6325 3575 50  0001 C CNN
 F 3 "" H 6325 3575 50  0000 C CNN
 	1    6325 3575
@@
 $EndComp
 $Comp
-L GND #PWR?
+L GND #PWR013
 U 1 1 59236587
 P 6325 3675
-F 0 "#PWR?" H 6325 3425 50  0001 C CNN
+F 0 "#PWR013" H 6325 3425 50  0001 C CNN
 F 1 "GND" H 6325 3525 50  0000 C CNN
 F 2 "" H 6325 3675 50  0000 C CNN
@@
 Connection ~ 6325 3400
 $Comp
-L C_Small C?
+L C_Small C2
 U 1 1 5923663D
 P 5900 3550
-F 0 "C?" H 5910 3620 50  0000 L CNN
+F 0 "C2" H 5910 3620 50  0000 L CNN
 F 1 "47nF" H 5910 3470 50  0000 L CNN
-F 2 "" H 5900 3550 50  0000 C CNN
+F 2 "Capacitors_SMD:C_0805_HandSoldering" H 5900 3550 50  0001 C CNN
 F 3 "" H 5900 3550 50  0000 C CNN
 	1    5900 3550
@@
 Connection ~ 5900 3400
 $Comp
-L C_Small C?
+L C_Small C1
 U 1 1 592366C6
 P 5575 3550
-F 0 "C?" H 5585 3620 50  0000 L CNN
+F 0 "C1" H 5585 3620 50  0000 L CNN
 F 1 "47nF" H 5585 3470 50  0000 L CNN
-F 2 "" H 5575 3550 50  0000 C CNN
+F 2 "Capacitors_SMD:C_0805_HandSoldering" H 5575 3550 50  0001 C CNN
 F 3 "" H 5575 3550 50  0000 C CNN
 	1    5575 3550
@@
 $EndComp
 $Comp
-L R_Small R?
+L R_Small R1
 U 1 1 592367A5
 P 5575 3750
-F 0 "R?" H 5605 3770 50  0000 L CNN
+F 0 "R1" H 5605 3770 50  0000 L CNN
 F 1 "150" H 5605 3710 50  0000 L CNN
-F 2 "" H 5575 3750 50  0000 C CNN
+F 2 "Resistors_SMD:R_0603_HandSoldering" H 5575 3750 50  0001 C CNN
 F 3 "" H 5575 3750 50  0000 C CNN
 	1    5575 3750
@@
 $EndComp
 $Comp
-L R_Small R?
+L R_Small R2
 U 1 1 59236850
 P 5900 3750
-F 0 "R?" H 5930 3770 50  0000 L CNN
+F 0 "R2" H 5930 3770 50  0000 L CNN
 F 1 "150" H 5930 3710 50  0000 L CNN
-F 2 "" H 5900 3750 50  0000 C CNN
+F 2 "Resistors_SMD:R_0603_HandSoldering" H 5900 3750 50  0001 C CNN
 F 3 "" H 5900 3750 50  0000 C CNN
 	1    5900 3750
