File: hardware/Rev2/MCU.sch (KiCad schematic (older format))
At the start: 23 parts

Commit message: created PCB and gerbers
Parts:
- removed JP? (x3): Jumper_NO_Small, symbol Jumper_NO_Small
- added C18, C19: 15uF 10v, Capacitors_SMD:C_1206_HandSoldering, symbol C_Small
- C10, C11, C4, C5, C6, C7, C8, C9: renamed from C?; footprint (none) -> Capacitors_SMD:C_0805_HandSoldering
- L1: renamed from L?; footprint (none) -> Resistors_SMD:R_1210_HandSoldering
- P1: renamed from P?; footprint (none) -> Pin_Headers:Pin_Header_Straight_2x03_Pitch2.54mm
- P2: renamed from P?; footprint (none) -> Pin_Headers:Pin_Header_Angled_1x06_Pitch2.54mm
- P3: renamed from P?; footprint (none) -> Pin_Headers:Pin_Header_Straight_2x04_Pitch2.54mm
- P4: renamed from P?; footprint (none) -> Pin_Headers:Pin_Header_Angled_1x03_Pitch2.54mm
- R3, R4, R5, R6, R7: renamed from R?; footprint (none) -> Resistors_SMD:R_0603_HandSoldering
- Y1: renamed from Y?; footprint (none) -> Crystals:Crystal_SMD_HC49-SD
- gave numbers to parts that had none: 1
Connections:
- net +3V3: now also C19.1
- net 5V: now also C18.1
- net CE: now also U4.10 ((PCINT22/OC0A/AIN0)PD6)
- net CSN: now also U4.9 ((PCINT21/OC0B/T1)PD5)
- net GND: now also C18.2, C19.2
- net IRQ: no longer U4.32 ((PCINT18/INT0)PD2)
- net MISO: now also P3.7 (P7)
- net MOSI: now also P3.6 (P6)
- net MRXSTX: now also U4.31 ((PCINT17/TXD)PD1); no longer U4.30 ((PCINT16/RXD)PD0)
- net MTXSRX: now also U4.30 ((PCINT16/RXD)PD0); no longer U4.31 ((PCINT17/TXD)PD1)
- net SCK: now also P3.5 (P5)
- net FET-drive: now reaches U4.1 ((PCINT19/OC2B/INT1)PD3)
